Commit message: can run rviz2

File: LAB2/src/sandevistan_description/robot/sandevistan.urdf (robot description, URDF)
Before this commit: robot sandevistan, 6 links, 1 joints
Links:
- added link end_effector
- link link_0: geometry visual mesh filename=package://sandevistan_description/meshes/link_0.STL
- link link_1: geometry visual mesh filename=package://sandevistan_description/meshes/link_1.STL
- link link_2: geometry visual mesh filename=package://sandevistan_description/meshes/link_2.STL
- link link_3: geometry visual mesh filename=package://sandevistan_description/meshes/link_3.STL
- link link_4: geometry visual mesh filename=package://sandevistan_description/meshes/link_4.STL
Joints:
- added joint joint_0: type revolute, parent link_0, child link_1, origin xyz=0 0 0.4 rpy=0 0 -1.57, axis 0 0 1, limit lower=-3.14 upper=3.14 effort=0.5 velocity=0.5
- added joint joint_1: type revolute, parent link_1, child link_2, origin xyz=0 0 0 rpy=-1.57 -1.57 0, axis 0 0 1, limit lower=-3.14 upper=3.14 effort=0.5 velocity=0.5
- added joint joint_2: type revolute, parent link_2, child link_3, origin xyz=0 -0.15 0 rpy=1.57 0 0, axis 0 0 1, limit lower=-3.14 upper=3.14 effort=0.5 velocity=0.5
- added joint joint_3: type prismatic, parent link_3, child link_4, origin xyz=0 0 0 rpy=0 0 0, axis 0 0 1, limit lower=0 upper=0.1 effort=0.5 velocity=0.5
- added joint joint_neff: type fixed, parent link_4, child end_effector, origin xyz=0 0 0 rpy=0 0 0, axis 0 0 0

Commit message: change joint axis pos and rotation

File: LAB2/src/sandevistan_description/robot/sandevistan.urdf (robot description, URDF)
Before this commit: robot sandevistan, 7 links, 6 joints
Joints:
- removed joint joint_0
- removed joint joint_1
- removed joint joint_2
- removed joint joint_3
- removed joint joint_base
- removed joint joint_neff
- added joint joint_0_1: type revolute, parent link_0, child link_1, origin xyz=0 0 0.4 rpy=0 0 -1.57, axis 0 0 1, limit lower=-3.14 upper=3.14 effort=0.5 velocity=0.5
- added joint joint_1_2: type revolute, parent link_1, child link_2, origin xyz=0 0 0 rpy=-1.57 -1.57 0, axis 0 0 1, limit lower=-3.14 upper=3.14 effort=0.5 velocity=0.5
- added joint joint_2_3: type revolute, parent link_2, child link_3, origin xyz=0 -0.15 0 rpy=1.57 0 0, axis 0 0 1, limit lower=-3.14 upper=3.14 effort=0.5 velocity=0.5
- added joint joint_3_4: type prismatic, parent link_3, child link_4, origin xyz=0 0 0 rpy=0 0 0, axis 0 0 1, limit lower=0 upper=0.1 effort=0.5 velocity=0.5
- added joint joint_4_neff: type fixed, parent link_4, child end_effector, origin xyz=0 0 0.2 rpy=3.14 -1.57 0, axis 0 0 0
- added joint joint_base_0: type fixed, parent base_link, child link_0, origin xyz=0 0 0 rpy=0 0 0, axis 0 0 0

Commit message: added code to kinematics server

File: LAB2/src/sandevistan_description/robot/sandevistan.urdf (robot description, URDF)
Before this commit: robot sandevistan, 7 links, 6 joints
Joints:
- joint joint_3_4: origin xyz=0 0 0 rpy=0 0 0 -> xyz=0 0 0.2 rpy=0 0 0
- joint joint_4_neff: origin xyz=0 0 0.2 rpy=3.14 -1.57 0 -> xyz=0 0 0 rpy=3.14 -1.57 0
