Commit message: xacro macros

File: LAB3/src/ros2_control_demo_3r_robot/description/example_robot.urdf.xacro (robot description, xacro)
@@ -4,8 +4,13 @@
     <!-- As we move through the file, new things to note will be pointed out. -->
     <!-- It's not meant an example of GOOD design, but an example of some of the various features of URDF/xacro. -->
+    <!-- Package Name -->
+    <xacro:property name="package" value="ros2_control_demo_3r_robot" />
     <!-- This will include all the contents of example_include.xacro first. Go check it out! -->
     <xacro:include filename="example_include.xacro" />
+    <xacro:include filename="create_link.xacro" />
+    <!-- Variables -->
+    <xacro:property name="pi" value="3.1415926535897931" />
     <!-- This first link called "world" is empty -->
-    <link name="world"></link>
+    <link name="world" />
     <!-- A simple fixed joint from our empty world link, to our base. -->
     <!-- The base origin is offset from the world origin. -->
@@ -15,34 +20,19 @@
         <child link="link_0"/>
     </joint>
-    <!-- base_link is a large rectangular plate. Some things to note: -->
-    <!-- - We set the visual origin Z to half the box height, so that the link origin sits at the bottom of the box -->
-    <!-- - We set the collision to be identical to the visual -->
-    <!-- - We specified the colour manually (but still need to enter a name) -->
-    <!-- - We specified all the inertial parameters manually -->
-    <link name="link_0">
-        <visual>
-            <origin xyz="0 0 0.0" rpy="0 0 0"/>
-            <geometry>
-                <!-- <box size="2.5 1.5 0.1" /> -->
-                <mesh filename="file:///$(find ros2_control_demo_3r_robot)/meshes/link_0.stl"/>
-            </geometry>
-            <material name="green">
-                <color rgba="0.2 1 0.2 1"/>
-            </material>
-        </visual>
-        <collision>
-            <origin xyz="0 0 0.0" rpy="0 0 0"/>
-            <contact_coefficients mu="0" kp="1000.0" kd="1.0"/>
-            <geometry>
-                <mesh filename="file:///$(find ros2_control_demo_3r_robot)/meshes/link_0.stl"/>
-                <!-- <box size="2.5 1.5 0.1" /> -->
-            </geometry>
-        </collision>
-        <inertial>
-            <origin xyz="0 0 0.05" rpy="0 0 0"/>
-            <mass value="120" />
-            <inertia ixx="0.001" ixy="0.0" ixz="0.0" iyy="0.001" iyz="0.0" izz="0.001" />
-        </inertial>
-    </link>
+    <xacro:addlink name="link_0">
+        <xacro:addvis>
+            <origin xyz="0 0 0" rpy="0 0 0"/>
+            <xacro:addmesh mesh_file="link_0.stl"/>
+            <xacro:addcolor color="idk" rgba="1.0 0.0 0.0 1.0"/>
+        </xacro:addvis>
+        <xacro:addcollide mu="0" kp="1000.0" kd="1.0">
+            <origin xyz="0 0 0" rpy="0 0 0"/>
+            <xacro:addmesh mesh_file="link_0.stl"/>
+        </xacro:addcollide>
+        <xacro:addinertia mass="100">
+            <origin xyz="0 0 0" rpy="0 0 0"/>
+            <inertia ixx="0.1" ixy="0.0" ixz="0.0" iyy="0.1" iyz="0.0" izz="0.1"/>
+        </xacro:addinertia>
+    </xacro:addlink>
     <joint name="joint_0" type="fixed">
         <parent link="link_0"/>
@@ -52,98 +42,69 @@
         <limit lower="-3.14" upper="3.14" effort="1000" velocity="0.5"/>
     </joint>
-    <link name="link_1">
-        <visual>
-            <origin xyz="0 0 0.0" rpy="0 0 0"/>
-            <geometry>
-                <!-- <box size="2.5 1.5 0.1" /> -->
-                <mesh filename="file:///$(find ros2_control_demo_3r_robot)/meshes/link_1.stl"/>
-            </geometry>
-            <material name="green">
-                <color rgba="0.2 1 0.2 1"/>
-            </material>
-        </visual>
-        <collision>
-            <origin xyz="0 0 0.0" rpy="0 0 0"/>
-            <contact_coefficients mu="0" kp="1000.0" kd="1.0"/>
-            <geometry>
-                <mesh filename="file:///$(find ros2_control_demo_3r_robot)/meshes/link_1.stl"/>
-                <!-- <box size="0.01 0.01 0.01" /> -->
-            </geometry>
-        </collision>
-        <inertial>
-            <origin xyz="0 0 0.0" rpy="0 0 0"/>
-            <mass value="25" />
+    <xacro:addlink name="link_1">
+        <xacro:addvis>
+            <origin xyz="0 0 0" rpy="0 0 0"/>
+            <xacro:addmesh mesh_file="link_1.stl"/>
+            <xacro:addcolor color="green" rgba="0.2 1 0.2 1.0"/>
+        </xacro:addvis>
+        <xacro:addcollide mu="0" kp="1000.0" kd="1.0">
+            <origin xyz="0 0 0" rpy="0 0 0"/>
+            <xacro:addmesh mesh_file="link_1.stl"/>
+        </xacro:addcollide>
+        <xacro:addinertia mass="25">
+            <origin xyz="0 0 0" rpy="0 0 0"/>
             <inertia ixx="0.001" ixy="0.0" ixz="0.0" iyy="0.001" iyz="0.0" izz="0.001" />
-        </inertial>
-    </link>
+        </xacro:addinertia>
+    </xacro:addlink>
     <joint name="joint_1" type="revolute">
         <parent link="link_0"/>
         <child link="link_1"/>
-        <origin rpy="0 0 0" xyz="0 0 0.16"/>
+        <origin rpy="0 0 0" xyz="0 0 0.1"/>
         <axis xyz="0 0 1"/>
         <limit lower="-3.14" upper="3.14" effort="1000" velocity="0.5"/>
         <dynamics damping="0" friction="0"/>
     </joint>
-    <link name="link_2">
-        <visual>
-            <origin xyz="0 0 0.0" rpy="0 0 0"/>
-            <geometry>
-                <!-- <box size="2.5 1.5 0.1" /> -->
-                <mesh filename="file:///$(find ros2_control_demo_3r_robot)/meshes/link_2.stl"/>
-            </geometry>
-            <material name="green">
-                <color rgba="0.2 1 0.2 1"/>
-            </material>
-        </visual>
-        <collision>
-            <contact_coefficients mu="0" kp="1000.0" kd="1.0"/>
-            <origin xyz="0 0 0.0" rpy="0 0 0"/>
-            <geometry>
-                <!-- <box size="0.01 0.01 0.01" /> -->
-                <mesh filename="file:///$(find ros2_control_demo_3r_robot)/meshes/link_2.stl"/>
-                <!-- <box size="2.5 1.5 0.1" /> -->
-            </geometry>
-        </collision>
-        <inertial>
-            <origin xyz="0 0 0.0" rpy="0 0 0"/>
-            <mass value="15" />
+    <xacro:addlink name="link_2">
+        <xacro:addvis>
+            <origin xyz="0 0 0" rpy="0 0 0"/>
+            <xacro:addmesh mesh_file="link_2.stl"/>
+            <xacro:addcolor color="green" rgba="0.2 1 0.2 1.0"/>
+        </xacro:addvis>
+        <xacro:addcollide mu="0" kp="1000.0" kd="1.0">
+            <origin xyz="0 0 0" rpy="0 0 0"/>
+            <xacro:addmesh mesh_file="link_2.stl"/>
+        </xacro:addcollide>
+        <xacro:addinertia mass="15">
+            <origin xyz="0 0 0" rpy="0 0 0"/>
             <inertia ixx="0.001" ixy="0.0" ixz="0.0" iyy="0.001" iyz="0.0" izz="0.001" />
-        </inertial>
-    </link>
+        </xacro:addinertia>
+    </xacro:addlink>
     <joint name="joint_2" type="revolute">
         <parent link="link_1"/>
         <child link="link_2"/>
-        <origin rpy="1.57079632679   0 0" xyz="0 0 0"/>
+        <origin rpy="${pi/2} 0 0" xyz="0 0 0"/>
         <axis xyz="0 0 1"/>
         <limit lower="-3.14" upper="3.14" effort="0.5" velocity="0.5"/>
         <dynamics damping="10" friction="10"/>
     </joint>
-    <link name="link_3">
-        <visual>
-            <origin xyz="0 0 0.0" rpy="0 0 0"/>
-            <geometry>
-                <mesh filename="file:///$(find ros2_control_demo_3r_robot)/meshes/link_3.stl"/>
-            </geometry>
-            <material name="green">
-                <color rgba="0.2 1 0.2 1"/>
-            </material>
-        </visual>
-        <collision>
-            <contact_coefficients mu="0" kp="1000.0" kd="1.0"/>
-            <origin xyz="0 0 0.0" rpy="0 0 0"/>
-            <geometry>
-                <mesh filename="file:///$(find ros2_control_demo_3r_robot)/meshes/link_3.stl"/>
-            </geometry>
-        </collision>
-        <inertial>
-            <origin xyz="0 0 0.0" rpy="0 0 0"/>
-            <mass value="5" />
+    <xacro:addlink name="link_3">
+        <xacro:addvis>
+            <origin xyz="0 0 0" rpy="0 0 0"/>
+            <xacro:addmesh mesh_file="link_3.stl"/>
+            <xacro:addcolor color="green" rgba="0.2 1 0.2 1.0"/>
+        </xacro:addvis>
+        <xacro:addcollide mu="0" kp="1000.0" kd="1.0">
+            <origin xyz="0 0 0" rpy="0 0 0"/>
+            <xacro:addmesh mesh_file="link_3.stl"/>
+        </xacro:addcollide>
+        <xacro:addinertia mass="5">
+            <origin xyz="0 0 0" rpy="0 0 0"/>
             <inertia ixx="0.001" ixy="0.0" ixz="0.0" iyy="0.001" iyz="0.0" izz="0.001" />
-        </inertial>
-    </link>
+        </xacro:addinertia>
+    </xacro:addlink>
     <joint name="joint_3" type="revolute">
         <parent link="link_2"/>
         <child link="link_3"/>
-        <origin rpy="0 0 0" xyz="0.37 0 0"/>
+        <origin rpy="0 0 0" xyz="0.15 0 0"/>
         <axis xyz="0 0 1"/>
         <limit lower="-3.14" upper="3.14" effort="1000" velocity="0.5"/>
@@ -156,6 +117,5 @@
         <axis xyz="0 0 1"/>
     </joint>
-    <link name="end_effector">
-    </link>
+    <link name="end_effector" />
     <xacro:include filename="example_gazebo.xacro" />
 </robot>
