Commit message: Updated LAB3

File: LAB3/install/ros2_control_demo_3r_robot/share/ros2_control_demo_3r_robot/description/create_link.xacro (robot description, xacro)
@@ -1 +1 @@
-/home/omzlette/gitROS/FRA333_LAB_HW/LAB3/src/ros2_control_demo_3r_robot/description/create_link.xacro
+/home/valdeus1151/Y3T1/FRA333_LAB_HW/LAB3/src/ros2_control_demo_3r_robot/description/create_link.xacro

File: LAB3/install/ros2_control_demo_3r_robot/share/ros2_control_demo_3r_robot/description/example_gazebo.xacro (robot description, xacro)
@@ -1 +1 @@
-/home/omzlette/gitROS/FRA333_LAB_HW/LAB3/src/ros2_control_demo_3r_robot/description/example_gazebo.xacro
+/home/valdeus1151/Y3T1/FRA333_LAB_HW/LAB3/src/ros2_control_demo_3r_robot/description/example_gazebo.xacro

File: LAB3/install/ros2_control_demo_3r_robot/share/ros2_control_demo_3r_robot/description/example_include.xacro (robot description, xacro)
@@ -1 +1 @@
-/home/omzlette/gitROS/FRA333_LAB_HW/LAB3/src/ros2_control_demo_3r_robot/description/example_include.xacro
+/home/valdeus1151/Y3T1/FRA333_LAB_HW/LAB3/src/ros2_control_demo_3r_robot/description/example_include.xacro

File: LAB3/install/ros2_control_demo_3r_robot/share/ros2_control_demo_3r_robot/description/example_robot.urdf.xacro (robot description, xacro)
@@ -1 +1 @@
-/home/omzlette/gitROS/FRA333_LAB_HW/LAB3/src/ros2_control_demo_3r_robot/description/example_robot.urdf.xacro
+/home/valdeus1151/Y3T1/FRA333_LAB_HW/LAB3/src/ros2_control_demo_3r_robot/description/example_robot.urdf.xacro

File: LAB3/src/ros2_control_demo_3r_robot/description/example_gazebo.xacro (robot description, xacro)
@@ -15,5 +15,5 @@
     <!-- This plugin will publish the joint_states for the selected joints
             (which robot_state_publisher can then use to broadcast the approprate tf). -->
-    <gazebo>
+    <!-- <gazebo>
         <plugin name="gazebo_ros_joint_state_publisher"
             filename="libgazebo_ros_joint_state_publisher.so">
@@ -23,5 +23,5 @@
             <joint_name>joint_3</joint_name>
         </plugin>
-    </gazebo>
+    </gazebo> -->
     <!-- This plugin will read a JointTrajectory message from the /set_joint_trajectory topic
             and move the machine accordingly. It's a bit clunky but it works. -->
@@ -45,4 +45,12 @@
                 <param name="max">3.14</param>
             </command_interface>
+            <command_interface name="velocity">
+                <param name="min">-10</param>
+                <param name="max">10</param>
+            </command_interface>
+            <command_interface name="effort">
+                <param name="min">-1000</param>
+                <param name="max">1000</param>
+            </command_interface>
             <state_interface name="position">
                 <param name="initial_value">0.0</param>
@@ -55,4 +63,12 @@
                 <param name="min">-3.14</param>
                 <param name="max">3.14</param>
+            </command_interface>
+            <command_interface name="velocity">
+                <param name="min">-10</param>
+                <param name="max">10</param>
+            </command_interface>
+            <command_interface name="effort">
+                <param name="min">-1000</param>
+                <param name="max">1000</param>
             </command_interface>
             <state_interface name="position">
@@ -67,4 +83,12 @@
                 <param name="max">3.14</param>
             </command_interface>
+            <command_interface name="velocity">
+                <param name="min">-10</param>
+                <param name="max">10</param>
+            </command_interface>
+            <command_interface name="effort">
+                <param name="min">-1000</param>
+                <param name="max">1000</param>
+            </command_interface>
             <state_interface name="position">
                 <param name="initial_value">0.0</param>
@@ -74,10 +98,10 @@
         </joint>
       </ros2_control>
-    <gazebo>
+    <!-- <gazebo>
         <plugin filename="libgazebo_ros2_control.so" name="gazebo_ros2_control">
             <robot_sim_type>gazebo_ros2_control/GazeboSystem</robot_sim_type>
           <parameters>$(find ros2_control_demo_3r_robot)/config/myrobot_controllers.yaml</parameters>
         </plugin>
-    </gazebo>
+    </gazebo> -->
     <gazebo reference="link0">
         <mu1>0.2</mu1>

File: LAB3/src/ros2_control_demo_3r_robot/description/example_robot.urdf.xacro (robot description, xacro)
@@ -26,20 +26,13 @@
             <xacro:addcolor color="idk" rgba="1.0 0.0 0.0 1.0"/>
         </xacro:addvis>
-        <xacro:addcollide mu="0" kp="1000.0" kd="1.0">
+        <xacro:addcollide mu="0" kp="10.0" kd="1.0">
             <origin xyz="0 0 0" rpy="0 0 0"/>
             <xacro:addmesh mesh_file="link_0.stl"/>
         </xacro:addcollide>
-        <xacro:addinertia mass="100">
-            <origin xyz="0 0 0" rpy="0 0 0"/>
-            <inertia ixx="0.1" ixy="0.0" ixz="0.0" iyy="0.1" iyz="0.0" izz="0.1"/>
+        <xacro:addinertia mass="0.310887">
+            <origin xyz="0 0 0.020724" rpy="0 0 0"/>
+            <inertia ixx="0.000222" ixy="0.0" ixz="0.0" iyy="0.000222" iyz="0.0" izz="0.000341"/>
         </xacro:addinertia>
     </xacro:addlink>
-    <joint name="joint_0" type="fixed">
-        <parent link="link_0"/>
-        <child link="link_1"/>
-        <origin rpy="0 0 0" xyz="0 0 0"/>
-        <axis xyz="0 0 1"/>
-        <limit lower="-3.14" upper="3.14" effort="1000" velocity="0.5"/>
-    </joint>
     <xacro:addlink name="link_1">
         <xacro:addvis>
@@ -48,11 +41,11 @@
             <xacro:addcolor color="green" rgba="0.2 1 0.2 1.0"/>
         </xacro:addvis>
-        <xacro:addcollide mu="0" kp="1000.0" kd="1.0">
+        <xacro:addcollide mu="0" kp="10.0" kd="1.0">
             <origin xyz="0 0 0" rpy="0 0 0"/>
             <xacro:addmesh mesh_file="link_1.stl"/>
         </xacro:addcollide>
-        <xacro:addinertia mass="25">
-            <origin xyz="0 0 0" rpy="0 0 0"/>
-            <inertia ixx="0.001" ixy="0.0" ixz="0.0" iyy="0.001" iyz="0.0" izz="0.001" />
+        <xacro:addinertia mass="0.204197">
+            <origin xyz="0 0 -0.048174" rpy="0 0 0"/>
+            <inertia ixx="0.000244" ixy="0.0" ixz="0.0" iyy="0.000238" iyz="0.0" izz="0.000082" />
         </xacro:addinertia>
     </xacro:addlink>
@@ -60,7 +53,7 @@
         <parent link="link_0"/>
         <child link="link_1"/>
-        <origin rpy="0 0 0" xyz="0 0 0.1"/>
+        <origin rpy="0 0 0" xyz="0 0 0.15"/>
         <axis xyz="0 0 1"/>
-        <limit lower="-3.14" upper="3.14" effort="1000" velocity="0.5"/>
+        <limit lower="${-pi}" upper="${pi}" effort="1" velocity="1"/>
         <dynamics damping="0" friction="0"/>
     </joint>
@@ -71,11 +64,11 @@
             <xacro:addcolor color="green" rgba="0.2 1 0.2 1.0"/>
         </xacro:addvis>
-        <xacro:addcollide mu="0" kp="1000.0" kd="1.0">
+        <xacro:addcollide mu="0" kp="10.0" kd="1.0">
             <origin xyz="0 0 0" rpy="0 0 0"/>
             <xacro:addmesh mesh_file="link_2.stl"/>
         </xacro:addcollide>
-        <xacro:addinertia mass="15">
-            <origin xyz="0 0 0" rpy="0 0 0"/>
-            <inertia ixx="0.001" ixy="0.0" ixz="0.0" iyy="0.001" iyz="0.0" izz="0.001" />
+        <xacro:addinertia mass="0.212044">
+            <origin xyz="0.0750 0 0" rpy="0 0 0"/>
+            <inertia ixx="0.000057" ixy="0.0" ixz="0.0" iyy="0.000586" iyz="0.0" izz="0.000620" />
         </xacro:addinertia>
     </xacro:addlink>
@@ -85,6 +78,6 @@
         <origin rpy="${pi/2} 0 0" xyz="0 0 0"/>
         <axis xyz="0 0 1"/>
-        <limit lower="-3.14" upper="3.14" effort="0.5" velocity="0.5"/>
-        <dynamics damping="10" friction="10"/>
+        <limit lower="0" upper="${pi}" effort="1" velocity="1"/>
+        <dynamics damping="0" friction="0"/>
     </joint>
     <xacro:addlink name="link_3">
@@ -94,11 +87,11 @@
             <xacro:addcolor color="green" rgba="0.2 1 0.2 1.0"/>
         </xacro:addvis>
-        <xacro:addcollide mu="0" kp="1000.0" kd="1.0">
+        <xacro:addcollide mu="0" kp="10.0" kd="1.0">
             <origin xyz="0 0 0" rpy="0 0 0"/>
             <xacro:addmesh mesh_file="link_3.stl"/>
         </xacro:addcollide>
-        <xacro:addinertia mass="5">
-            <origin xyz="0 0 0" rpy="0 0 0"/>
-            <inertia ixx="0.001" ixy="0.0" ixz="0.0" iyy="0.001" iyz="0.0" izz="0.001" />
+        <xacro:addinertia mass="0.199772">
+            <origin xyz="0.044973 0 0" rpy="0 0 0"/>
+            <inertia ixx="0.000088" ixy="0.0" ixz="0.0" iyy="0.000211" iyz="0.0" izz="0.000202" />
         </xacro:addinertia>
     </xacro:addlink>
@@ -108,6 +101,6 @@
         <origin rpy="0 0 0" xyz="0.15 0 0"/>
         <axis xyz="0 0 1"/>
-        <limit lower="-3.14" upper="3.14" effort="1000" velocity="0.5"/>
-        <dynamics damping="10" friction="10"/>
+        <limit lower="${-pi/2}" upper="${pi/2}" effort="1" velocity="1"/>
+        <dynamics damping="0" friction="0"/>
     </joint>
     <joint name="joint_eff" type="fixed">
