Commit message: Updated LAB3

File: LAB3/src/fra333_lab3_29_v1/sandevistan_description/xacro_description/sandevistan_robot.urdf.xacro (robot description, xacro)
@@ -56,5 +56,5 @@
         <origin rpy="0 0 0" xyz="0 0 0.15"/>
         <axis xyz="0 0 1"/>
-        <limit lower="${-pi}" upper="${pi}" effort="1" velocity="1"/>
+        <limit lower="${-pi*2}" upper="${pi*2}" effort="1" velocity="1"/>
         <dynamics damping="0" friction="0"/>
     </joint>
