Commit message: Updated LAB4

File: LAB4/src/lab4_29/doppelt_description/xacro/doppelt_robot.urdf.xacro (robot description, xacro)
@@ -102,5 +102,5 @@
         <origin rpy="0 0 0" xyz="0.15 0 0"/>
         <axis xyz="0 0 1"/>
-        <limit lower="${-pi/2}" upper="${pi/2}" effort="1" velocity="1"/>
+        <limit lower="${-5*pi/6}" upper="${5*pi/6}" effort="1" velocity="1"/>
         <dynamics damping="0" friction="0"/>
     </joint>
@@ -108,5 +108,5 @@
         <parent link="link_3"/>
         <child link="end_effector"/>
-        <origin rpy="1.57 0 1.57" xyz="0.26 0 0"/>
+        <origin rpy="-1.57 0 0" xyz="0.2 0 0"/>
         <axis xyz="0 0 1"/>
     </joint>

Commit message: Updated Launch and URDF

File: LAB4/src/lab4_29/doppelt_description/xacro/doppelt_robot.urdf.xacro (robot description, xacro)
@@ -92,7 +92,7 @@
             <xacro:addmesh mesh_file="link_3.stl"/>
         </xacro:addcollide>
-        <xacro:addinertia mass="0.199772">
-            <origin xyz="0.044973 0 0" rpy="0 0 0"/>
-            <inertia ixx="0.000088" ixy="0.0" ixz="0.0" iyy="0.000211" iyz="0.0" izz="0.000202" />
+        <xacro:addinertia mass="0.314355">
+            <origin xyz="0.101895 0 0" rpy="0 0 0"/>
+            <inertia ixx="0.000155" ixy="0.0" ixz="0.0" iyy="0.001167" iyz="0.0" izz="0.001141" />
         </xacro:addinertia>
     </xacro:addlink>

Commit message: fix pi controller

File: LAB4/src/lab4_29/doppelt_description/xacro/doppelt_robot.urdf.xacro (robot description, xacro)
@@ -16,9 +16,4 @@
     <!-- A simple fixed joint from our empty world link, to our base. -->
     <!-- The base origin is offset from the world origin. -->
-    <joint name="base_joint" type="fixed">
-        <origin xyz="0 0 0" rpy="0 0 0"/>
-        <parent link="world"/>
-        <child link="link_0"/>
-    </joint>
     <xacro:addlink name="link_0">
         <xacro:addvis>
@@ -36,4 +31,9 @@
         </xacro:addinertia>
     </xacro:addlink>
+    <joint name="base_joint" type="fixed">
+        <origin xyz="0 0 0" rpy="0 0 0"/>
+        <parent link="world"/>
+        <child link="link_0"/>
+    </joint>
     <xacro:addlink name="link_1">
         <xacro:addvis>
@@ -105,4 +105,5 @@
         <dynamics damping="0" friction="0"/>
     </joint>
+    <link name="end_effector" />
     <joint name="joint_eff" type="fixed">
         <parent link="link_3"/>
@@ -111,4 +112,3 @@
         <axis xyz="0 0 1"/>
     </joint>
-    <link name="end_effector" />
 </robot>
